Commit message: Capticalize STL file names

File: fanuc_r2000ic_support/urdf/r2000ic125l_macro.xacro (robot description, xacro)
@@ -8,5 +8,5 @@
         <origin xyz="0 0 0" rpy="0 0 0"/>
         <geometry>
-          <mesh filename="package://fanuc_r2000ic_support/meshes/r2000ic125l/visual/base_link.stl" />
+          <mesh filename="package://fanuc_r2000ic_support/meshes/r2000ic125l/visual/base_link.STL" />
         </geometry>
         <xacro:material_fanuc_gray40 />
@@ -15,5 +15,5 @@
         <origin xyz="0 0 0" rpy="0 0 0"/>
         <geometry>
-          <mesh filename="package://fanuc_r2000ic_support/meshes/r2000ic125l/collision/base_link.stl" />
+          <mesh filename="package://fanuc_r2000ic_support/meshes/r2000ic125l/collision/base_link.STL" />
         </geometry>
       </collision>
@@ -37,12 +37,12 @@
         <origin xyz="0 0 0" rpy="0 0 0"/>
         <geometry>
-          <mesh filename="package://fanuc_r2000ic_support/meshes/r2000ic125l/visual/link_1.stl" />
-        </geometry>
-        <xacro:material_fanuc_yellow />
-      </visual>
-      <collision>
-        <origin xyz="0 0 0" rpy="0 0 0"/>
-        <geometry>
-          <mesh filename="package://fanuc_r2000ic_support/meshes/r2000ic125l/collision/link_1.stl" />
+          <mesh filename="package://fanuc_r2000ic_support/meshes/r2000ic125l/visual/link_1.STL" />
+        </geometry>
+        <xacro:material_fanuc_yellow />
+      </visual>
+      <collision>
+        <origin xyz="0 0 0" rpy="0 0 0"/>
+        <geometry>
+          <mesh filename="package://fanuc_r2000ic_support/meshes/r2000ic125l/collision/link_1.STL" />
         </geometry>
       </collision>
@@ -66,12 +66,12 @@
         <origin xyz="0 0 0" rpy="0 0 0"/>
         <geometry>
-          <mesh filename="package://fanuc_r2000ic_support/meshes/r2000ic125l/visual/link_2.stl" />
-        </geometry>
-        <xacro:material_fanuc_yellow />
-      </visual>
-      <collision>
-        <origin xyz="0 0 0" rpy="0 0 0"/>
-        <geometry>
-          <mesh filename="package://fanuc_r2000ic_support/meshes/r2000ic125l/collision/link_2.stl" />
+          <mesh filename="package://fanuc_r2000ic_support/meshes/r2000ic125l/visual/link_2.STL" />
+        </geometry>
+        <xacro:material_fanuc_yellow />
+      </visual>
+      <collision>
+        <origin xyz="0 0 0" rpy="0 0 0"/>
+        <geometry>
+          <mesh filename="package://fanuc_r2000ic_support/meshes/r2000ic125l/collision/link_2.STL" />
         </geometry>
       </collision>
@@ -95,12 +95,12 @@
         <origin xyz="0 0 0" rpy="0 0 0"/>
         <geometry>
-          <mesh filename="package://fanuc_r2000ic_support/meshes/r2000ic125l/visual/link_3.stl" />
-        </geometry>
-        <xacro:material_fanuc_yellow />
-      </visual>
-      <collision>
-        <origin xyz="0 0 0" rpy="0 0 0"/>
-        <geometry>
-          <mesh filename="package://fanuc_r2000ic_support/meshes/r2000ic125l/collision/link_3.stl" />
+          <mesh filename="package://fanuc_r2000ic_support/meshes/r2000ic125l/visual/link_3.STL" />
+        </geometry>
+        <xacro:material_fanuc_yellow />
+      </visual>
+      <collision>
+        <origin xyz="0 0 0" rpy="0 0 0"/>
+        <geometry>
+          <mesh filename="package://fanuc_r2000ic_support/meshes/r2000ic125l/collision/link_3.STL" />
         </geometry>
       </collision>
@@ -124,12 +124,12 @@
         <origin xyz="0 0 0" rpy="0 0 0"/>
         <geometry>
-          <mesh filename="package://fanuc_r2000ic_support/meshes/r2000ic125l/visual/link_4.stl" />
-        </geometry>
-        <xacro:material_fanuc_yellow />
-      </visual>
-      <collision>
-        <origin xyz="0 0 0" rpy="0 0 0"/>
-        <geometry>
-          <mesh filename="package://fanuc_r2000ic_support/meshes/r2000ic125l/collision/link_4.stl" />
+          <mesh filename="package://fanuc_r2000ic_support/meshes/r2000ic125l/visual/link_4.STL" />
+        </geometry>
+        <xacro:material_fanuc_yellow />
+      </visual>
+      <collision>
+        <origin xyz="0 0 0" rpy="0 0 0"/>
+        <geometry>
+          <mesh filename="package://fanuc_r2000ic_support/meshes/r2000ic125l/collision/link_4.STL" />
         </geometry>
       </collision>
@@ -153,12 +153,12 @@
         <origin xyz="0 0 0" rpy="0 0 0"/>
         <geometry>
-          <mesh filename="package://fanuc_r2000ic_support/meshes/r2000ic125l/visual/link_5.stl" />
-        </geometry>
-        <xacro:material_fanuc_yellow />
-      </visual>
-      <collision>
-        <origin xyz="0 0 0" rpy="0 0 0"/>
-        <geometry>
-          <mesh filename="package://fanuc_r2000ic_support/meshes/r2000ic125l/collision/link_5.stl" />
+          <mesh filename="package://fanuc_r2000ic_support/meshes/r2000ic125l/visual/link_5.STL" />
+        </geometry>
+        <xacro:material_fanuc_yellow />
+      </visual>
+      <collision>
+        <origin xyz="0 0 0" rpy="0 0 0"/>
+        <geometry>
+          <mesh filename="package://fanuc_r2000ic_support/meshes/r2000ic125l/collision/link_5.STL" />
         </geometry>
       </collision>
@@ -182,5 +182,5 @@
         <origin xyz="0 0 0" rpy="0 0 0"/>
         <geometry>
-          <mesh filename="package://fanuc_r2000ic_support/meshes/r2000ic125l/visual/link_6.stl" />
+          <mesh filename="package://fanuc_r2000ic_support/meshes/r2000ic125l/visual/link_6.STL" />
         </geometry>
         <xacro:material_fanuc_black />
@@ -189,5 +189,5 @@
         <origin xyz="0 0 0" rpy="0 0 0"/>
         <geometry>
-          <mesh filename="package://fanuc_r2000ic_support/meshes/r2000ic125l/collision/link_6.stl" />
+          <mesh filename="package://fanuc_r2000ic_support/meshes/r2000ic125l/collision/link_6.STL" />
         </geometry>
       </collision>
